File: board/board.kicad_pcb (KiCad board)
At the start: 2 copper layers, 91.5 x 68.6 mm, 66 parts, among them J1 Conn_01x25_Socket, J2 Conn_01x01, J2 Conn_01x25_Socket, J3 Conn_01x01, J4 Conn_01x01, J5 Conn_01x01, J5 PJ-320B, J6 Screw_Terminal_01x02, J7 Screw_Terminal_01x02, J8 Screw_Terminal_01x02

Commit message: attempt at tracing v2
Parts:
- removed H1: MountingHole, MountingHole:MountingHole_3.2mm_M3
- removed the J3 at (111.0, 57.0)
- removed the J4 at (111.0, 52.0)
- added C24: 0.22uF_0603_25V, 4ms_Capacitor:C_0603, F.Cu at (152.2, 61.4)
- added C25: 0.22uF_0603_25V, 4ms_Capacitor:C_0603, F.Cu at (152.2, 68.8)
- added J1: ~, TestPoint:TestPoint_Keystone_5019_Minature, F.Cu at (155.0, 91.1)
- added J2: ~, TestPoint:TestPoint_Keystone_5019_Minature, F.Cu at (150.8, 91.1)
- C13, C4, C8: value 0.22uF_0603_25V -> 22uF_0603_16V; footprint 4ms_Capacitor:C_0603 -> 4ms_Capacitor:C_0805
- C14, C18, C21, C9: value 0.22uF_0603_25V -> 22uF_0603_16V; footprint 4ms_Capacitor:C_0603 -> 4ms_Capacitor:C_0805; moved to F.Cu
- C15, C2, C22, C3, C5, C6, U2: moved to B.Cu
- C23, R15: moved to F.Cu
- R1, R2, R6: value 3.0k_0603_0.1% -> 100k_0603
- R11: value 100k_0603 -> 3.0k_0603_0.1%; moved to F.Cu
- R12, R14: value 100k_0603 -> 1k_0603_0.1%
- R13: value 1k_0603_0.1% -> 3.0k_0603_0.1%; moved to F.Cu
- R8: value 1k_0603_0.1% -> 2.2k_0603
- R9: value 2.2k_0603 -> 3.0k_0603_0.1%
- U1: footprint Package_SO:SOIC-8_3.9x4.9mm_P1.27mm -> project:AD9833
- U11: footprint 4ms_Package_DIP:DIP-8pin_TH -> project:W25Q128_board
- U12: footprint project:W25Q128_board -> Package_SO:SOIC-16W_7.5x10.3mm_P1.27mm
- U13: footprint 4ms_Package_DIP:DIP-8pin_TH -> Package_SO:SOIC-8_3.9x4.9mm_P1.27mm
- U14: footprint Package_SO:SOIC-16W_7.5x10.3mm_P1.27mm -> 4ms_Package_DIP:DIP-8pin_TH; moved to B.Cu
- U5: footprint project:AD9833 -> Package_SO:VSSOP-10_3x3mm_P0.5mm; moved to F.Cu
- U7: footprint Package_SO:VSSOP-10_3x3mm_P0.5mm -> 4ms_Package_DIP:DIP-8pin_TH
- moved G*** 103.6 mm to (73.0, 86.0)
- moved R11 90.2 mm to (227.8, 103.0), turned to 0 degrees
- moved R15 84.8 mm to (227.8, 113.2), turned to 0 degrees
- moved R13 81.6 mm to (227.8, 108.1), turned to 0 degrees
- moved R5 75.5 mm to (219.3, 113.2)
- moved R3 72.5 mm to (219.3, 108.1)
- moved R4 72.3 mm to (219.3, 110.6)
- moved R7 71.3 mm to (223.6, 105.5)
- moved C23 69.6 mm to (209.0, 86.0)
- moved U11 68.4 mm to (165.0, 57.1), turned to -90 degrees
- moved R8 68.1 mm to (223.6, 108.1), turned to 0 degrees
- moved R9 66.8 mm to (223.6, 110.6), turned to 0 degrees
- moved R10 65.7 mm to (223.6, 113.2), turned to 0 degrees
- moved C8 62.5 mm to (113.2, 73.2), turned to 90 degrees
- moved U13 60.6 mm to (211.0, 92.0)
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- renumbered J1 to J3, J2 to J4
Connections:
- C10 pad 1: P,-15 -> P,+15
- C11 pad 1: P,+15 -> +5V
- C13 pad 1: +3.3V -> Net-(U9-VinL)
- C13 pad 2: GND -> CH3_TOVOL
- C14 pad 1: +5V -> Net-(U10-VinR)
- C14 pad 2: GND -> NOISE_TOVOL
- C15 pad 1: +5V -> P,+15
- C16 pad 1: P,+15 -> +5V
- C18 pad 1: +5V -> Net-(U12-VinR)
- C18 pad 2: GND -> DAC_tovol1
- C20 pad 1: P,-15 -> +5V
- C21 pad 1: P,-5 -> Net-(U12-VinL)
- C21 pad 2: GND -> DAC_tovol2
- C22 pad 1: +5V -> P,-15
- C4 pad 1: +5V -> Net-(U8-VinR)
- C4 pad 2: GND -> CH2_TOVOL
- C6 pad 1: +5V -> P,+15
- C7 pad 1: +5V -> P,-15
- C8 pad 1: +5V -> Net-(U8-VinL)
- C8 pad 2: GND -> CH1_TOVOL
- C9 pad 1: P,+15 -> Net-(U9-VinR)
- C9 pad 2: GND -> CH4_TOVOL
- J3 pad 19: NOISE_CLK_SEL -> /PB2
- J4 pad 16: /PC1 -> NOISE_CLK_SEL
- J5 pad 1: Net-(U1-OUT_A) -> Net-(U13-OUT_A)
- J5 pad 2: Net-(U1-OUT_A) -> Net-(U13-OUT_A)
- R1 pad 1: CH1_OUT -> GND
- R1 pad 2: Net-(U1-IN_A) -> Analog_data_out1
- R10 pad 1: Net-(U1-IN_A) -> Net-(U13-INV_IN_A)
- R11 pad 1: GND -> DAC_out1
- R11 pad 2: Analog_data_out1 -> Net-(U13-IN_A)
- R12 pad 1: GND -> FILTER_FEEDBACK_OUT
- R12 pad 2: Analog_data_out2 -> Net-(U14-Vin)
- R13 pad 1: FILTER_FEEDBACK_OUT -> DAC_out2
- R13 pad 2: Net-(U13-Vin) -> Net-(U13-IN_A)
- R14 pad 1: GND -> Net-(U14-Vin)
- R14 pad 2: Analog_data_out3 -> CH4_TOFILT
- R15 pad 1: Net-(U13-Vin) -> Net-(U13-IN_A)
- R15 pad 2: CH4_TOFILT -> GND
- R2 pad 1: CH2_OUT -> GND
- R2 pad 2: Net-(U1-IN_A) -> Analog_data_out2
- R3 pad 1: CH3_OUT -> CH1_OUT
- R3 pad 2: Net-(U1-IN_A) -> Net-(U13-IN_A)
- R4 pad 1: CH4_OUT -> CH2_OUT
- R4 pad 2: Net-(U1-IN_A) -> Net-(U13-IN_A)
- R5 pad 1: NOISE_OUT -> CH3_OUT
- R5 pad 2: Net-(U1-IN_A) -> Net-(U13-IN_A)
- R6 pad 1: DAC_out1 -> GND
- R6 pad 2: Net-(U1-IN_A) -> Analog_data_out3
- R7 pad 1: DAC_out2 -> CH4_OUT
- R7 pad 2: Net-(U1-IN_A) -> Net-(U13-IN_A)
- R8 pad 1: Net-(U1-INV_IN_A) -> Net-(U13-OUT_A)
- R8 pad 2: GND -> Net-(U13-INV_IN_A)
- R9 pad 1: Net-(U1-OUT_A) -> NOISE_OUT
- R9 pad 2: Net-(U1-INV_IN_A) -> Net-(U13-IN_A)
- U1 pad 1: Net-(U1-OUT_A) -> +5V
- U1 pad 2: Net-(U1-INV_IN_A) -> GND
- U1 pad 3: Net-(U1-IN_A) -> Analog_data
- U1 pad 4: GND -> Analog_CLK
- U1 pad 5: unconnected-(U1-IN_B-Pad5) -> CS_AD9833_1
- U1 pad 6: unconnected-(U1-INV_IN_B-Pad6) -> GND
- U1 pad 7: unconnected-(U1-OUT_B-Pad7) -> DDS1_out
- U10 pad 9: NOISE_TOVOL -> Net-(U10-VinR)
- U11 pad 1: NOISE_TOVOL -> +3.3V
- U11 pad 2: unconnected-(U11-NC-Pad2) -> FLASH_CS
- U11 pad 3: +5V -> FLASH_MISO
- U11 pad 5: NOISE_DI -> FLASH_CLK
- U11 pad 6: NOISE_CS -> FLASH_MOSI
- U12 pad 1: +3.3V -> ZCEN_DAC
- U12 pad 2: FLASH_CS -> ATTEN_CS
- U12 pad 3: FLASH_MISO -> Analog_data_out3
- U12 pad 4: GND -> +5V
- U12 pad 5: FLASH_CLK -> GND
- U12 pad 6: FLASH_MOSI -> Analog_CLK
- U13 pad 1: Net-(U13-Vin) -> Net-(U13-OUT_A)
- U13 pad 2: GND -> Net-(U13-INV_IN_A)
- U13 pad 3: P,-5 -> Net-(U13-IN_A)
- U13 pad 4: unconnected-(U13-CLK_OUT-Pad4) -> GND
- U13 pad 5: FILT_CLK -> unconnected-(U13-IN_B-Pad5)
- U13 pad 6: +5V -> unconnected-(U13-INV_IN_B-Pad6)
- U13 pad 7: CH4_OUT -> unconnected-(U13-OUT_B-Pad7)
- U13 pad 8: GND -> +5V
- U14 pad 1: ZCEN_DAC -> Net-(U14-Vin)
- U14 pad 2: ATTEN_CS -> GND
- U14 pad 3: Analog_data_out3 -> P,-5
- U14 pad 4: +5V -> unconnected-(U14-CLK_OUT-Pad4)
- U14 pad 5: GND -> FILT_CLK
- U14 pad 6: Analog_CLK -> +5V
- U14 pad 7: unconnected-(U14-SDO-Pad7) -> CH4_OUT
- U14 pad 8: +5V -> GND
- U4 pad 5: CS_AD9833_1 -> CS_AD9833_4
- U4 pad 7: DDS1_out -> DDS4_out
- U5 pad 1: +5V -> MUX_SEL_1
- U5 pad 2: GND -> PWM2
- U5 pad 3: Analog_data -> GND
- U5 pad 4: Analog_CLK -> PWM1
- U5 pad 5: CS_AD9833_4 -> MUX_SEL_2
- U5 pad 6: GND -> CH1_TOVOL
- U5 pad 7: DDS4_out -> DDS1_out
- U6 pad 1: MUX_SEL_1 -> MUX_SEL_4
- U6 pad 10: CH1_TOVOL -> CH4_TOVOL
- U6 pad 2: DDS1_out -> PWM4
- U6 pad 4: DDS2_out -> PWM3
- U6 pad 5: MUX_SEL_2 -> MUX_SEL_3
- U6 pad 6: CH2_TOVOL -> CH3_TOVOL
- U6 pad 7: PWM2 -> DDS3_out
- U6 pad 9: PWM1 -> DDS4_out
- U7 pad 1: MUX_SEL_4 -> NOISE_TOVOL
- U7 pad 2: PWM4 -> unconnected-(U7-NC-Pad2)
- U7 pad 3: GND -> +5V
- U7 pad 4: PWM3 -> GND
- U7 pad 5: MUX_SEL_3 -> NOISE_DI
- U7 pad 6: CH3_TOVOL -> NOISE_CS
- U7 pad 7: DDS3_out -> NOISE_CLK
- U7 pad 8: +5V -> NOISE_CLK_SEL
- U8 pad 16: CH1_TOVOL -> Net-(U8-VinL)
- U8 pad 9: CH2_TOVOL -> Net-(U8-VinR)
- U9 pad 16: CH3_TOVOL -> Net-(U9-VinL)
- U9 pad 9: CH4_TOVOL -> Net-(U9-VinR)
Routing:
- net +5V: track 305.3 -> 64.1 mm, vias 38 -> 6
- net P,+15: track 125.3 -> 11.9 mm, vias 19 -> 4
- net P,-15: track 116.3 -> 11.9 mm, vias 20 -> 4
- net Analog_CLK: track 113.3 -> 16.0 mm, vias 6 -> 0
- net ATTEN_CS: track 97.1 -> 0.00 mm, vias 6 -> 0
- net DAC_tovol2: track 98.1 -> 4.02 mm
- net DAC_tovol1: track 96.8 -> 4.12 mm
- net CS_AD9833_2: track 78.8 -> 0.00 mm
- net NOISE_CS: track 75.7 -> 0.00 mm
- net PWM1: track 73.3 -> 0.00 mm
- net NOISE_CLK: track 68.8 -> 0.00 mm, vias 5 -> 0
- net NOISE_DI: track 66.3 -> 0.00 mm, vias 3 -> 0
- net Analog_data: track 70.5 -> 10.9 mm, vias 4 -> 0
- net PWM3: track 57.3 -> 0.00 mm, vias 7 -> 0
- net ZCEN_1: track 56.1 -> 0.00 mm, vias 3 -> 0
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- removed copper zone on B.Cu, net GND
- removed copper zone on F.Cu, net GND
Other:
- board text added: "PA8"
- board text removed: "DAC out"
- board text removed: "PA8 (clock)"

Commit message: W I D E
Other:
- board size 91.5 x 68.6 mm -> 92 x 75.8 mm
Changed lines of the file:
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@@
 	)
 	(gr_line
-		(start 98.270142 58.000001)
-		(end 107.220177 58.000001)
+		(start 98.2 58.000001)
+		(end 107.150035 58.000001)
 		(stroke
 			(width 0.1)
@@
 	)
 	(gr_line
-		(start 98.330142 106.92)
-		(end 98.350142 117.08)
-		(stroke
-			(width 0.1)
-			(type default)
-		)
-		(layer "Edge.Cuts")
-	)
-	(gr_line
-		(start 189.770142 117.08)
-		(end 189.770142 48.5)
+		(start 97.98 107)
+		(end 98 121)
+		(stroke
+			(width 0.1)
+			(type default)
+		)
+		(layer "Edge.Cuts")
+	)
+	(gr_line
+		(start 190 121)
+		(end 190 45.2)
 		(stroke
 			(width 0.1)
@@
 	)
 	(gr_line
-		(start 107.220142 58.025)
-		(end 107.220142 106.92)
-		(stroke
-			(width 0.1)
-			(type default)
-		)
-		(layer "Edge.Cuts")
-	)
-	(gr_line
-		(start 98.270142 48.5)
-		(end 189.770142 48.5)
+		(start 107.220177 58.000001)
+		(end 107.2 107)
+		(stroke
+			(width 0.1)
+			(type default)
+		)
+		(layer "Edge.Cuts")
+	)
+	(gr_line
+		(start 98.2 45.2)
+		(end 190 45.2)
 		(stroke
 			(width 0.1)
@@
 	)
 	(gr_line
-		(start 107.220142 106.92)
-		(end 98.330142 106.92)
-		(stroke
-			(width 0.1)
-			(type default)
-		)
-		(layer "Edge.Cuts")
-	)
-	(gr_line
-		(start 189.770142 117.08)
-		(end 98.350142 117.08)
-		(stroke
-			(width 0.1)
-			(type default)
-		)
-		(layer "Edge.Cuts")
-	)
-	(gr_line
-		(start 98.270142 48.5)
-		(end 98.270142 58.000001)
+		(start 107.2 107)
+		(end 98.11 107)
+		(stroke
+			(width 0.1)
+			(type default)
+		)
+		(layer "Edge.Cuts")
+	)
+	(gr_line
+		(start 190 121)
+		(end 98 121)
+		(stroke
+			(width 0.1)
+			(type default)
+		)
+		(layer "Edge.Cuts")
+	)
+	(gr_line
+		(start 98.2 45.2)
+		(end 98.2 58.000001)
 		(stroke
 			(width 0.1)
@@
 	)
 	(gr_text "PB5"
-		(at 159.35 51.9 90)
+		(at 159.2 51 90)
 		(layer "F.SilkS")
 		(effects
@@
 	)
 	(gr_text "PD2"
-		(at 166.85 52 90)
+		(at 166.85 51 90)
 		(layer "F.SilkS")
 		(effects
@@
 	)
 	(gr_text "PC9"
-		(at 159.35 116.95 90)
+		(at 159.35 118 90)
 		(layer "F.SilkS")
 		(effects
@@
 	)
 	(gr_text "PB4"
-		(at 161.75 51.9 90)
+		(at 161.75 51 90)
 		(layer "F.SilkS")
 		(effects
@@
 	)
 	(gr_text "PB14"
-		(at 146.5 117.15 90)
+		(at 146.5 119 90)
 		(layer "F.SilkS")
 		(effects
@@
 	)
 	(gr_text "PC7"
-		(at 154.3 116.95 90)
+		(at 154.3 118 90)
 		(layer "F.SilkS")
 		(effects
@@
 	)
 	(gr_text "PC6"
-		(at 151.7 116.95 90)
+		(at 151.7 118 90)
 		(layer "F.SilkS")
 		(effects
@@
 	)
 	(gr_text "PB6"
-		(at 156.7 51.9 90)
+		(at 156.7 51 90)
 		(layer "F.SilkS")
 		(effects
@@
 	)
 	(gr_text "PB15"
-		(at 149.15 117.1 90)
+		(at 149 119 90)
 		(layer "F.SilkS")
 		(effects
@@
 	)
 	(gr_text "PC12"
-		(at 169.4 52.55 90)
+		(at 169.4 51 90)
 		(layer "F.SilkS")
 		(effects
@@
 	)
 	(gr_text "PA15"
-		(at 171.95 52.4 90)
+		(at 171.95 51 90)
 		(layer "F.SilkS")
 		(effects
@@
 	)
 	(gr_text "PC8"
-		(at 156.7 116.95 90)
+		(at 156.7 118 90)
 		(layer "F.SilkS")
 		(effects
@@
 	)
 	(gr_text "PB3"
-		(at 164.3 51.9 90)
-		(layer "F.SilkS")
-		(effects
+		(at 164.3 51 90)
+		(layer "F.SilkS")
+		(effects

Commit message: more tracing...
Parts:
- moved R13 59.3 mm to (169.7, 96.0)
- moved R11 59.0 mm to (169.7, 93.0)
- moved R15 58.1 mm to (171.4, 99.2)
- moved R3 58.0 mm to (169.7, 78.0)
- moved R4 57.8 mm to (169.7, 81.0)
- moved R9 57.7 mm to (169.7, 90.0)
- moved R5 57.5 mm to (169.7, 84.0)
- moved R7 57.0 mm to (169.7, 87.0)
- moved R10 56.1 mm to (174.9, 85.2), turned to 180 degrees
- moved R8 49.1 mm to (180.0, 85.2), turned to 180 degrees
- moved U13 36.2 mm to (176.7, 80.4), turned to 0 degrees
- moved C23 27.4 mm to (182.7, 78.4), turned to 0 degrees
- moved J6 22.1 mm to (208.0, 76.5)
- moved J7 22.1 mm to (208.0, 86.5)
- moved J8 22.1 mm to (208.0, 96.5)
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Routing:
- net Net-(U13-IN_A): track 0.00 -> 24.9 mm
- net Net-(U13-OUT_A): track 8.33 -> 31.7 mm
- net Net-(U13-INV_IN_A): track 0.00 -> 10.2 mm
- net +3.3V: track 0.00 -> 9.70 mm
- net +5V: track 64.1 -> 66.8 mm
- net DAC_tovol1: track 4.12 -> 3.28 mm
