File: board/boardv3_morning01112024.kicad_pcb (KiCad board)
At the start: 2 copper layers, 92 x 75.8 mm, 69 parts, among them J2 Conn_01x01, J3 Conn_01x01, J3 Conn_01x25_Socket, J4 Conn_01x01, J4 Conn_01x25_Socket, J5 Conn_01x01, J5 PJ-320B, J6 Screw_Terminal_01x02, J7 Screw_Terminal_01x02, J8 Screw_Terminal_01x02

Commit message: hopefully final PCB
Parts:
- removed the G*** at (121.3, 99.5)
- added G***: LOGO, project:logo_negative, F.Cu at (119.2, 100.0)
- C23: moved to B.Cu
- moved C23 0.81 mm to (176.3, 74.5)
Routing:
- net P,-15: track 132.4 -> 125.7 mm, vias 7 -> 9
- net CS_AD9833_1: track 48.7 -> 43.7 mm
- net CS_AD9833_3: track 49.0 -> 46.4 mm
- net CS_AD9833_4: track 57.8 -> 55.8 mm
- net CH2_OUT: track 70.0 -> 71.3 mm
- net +5V: track 259.5 -> 260.7 mm, vias 8 -> 9
- net Analog_data: track 75.7 -> 76.3 mm
- net CS_AD9833_2: track 64.0 -> 63.4 mm
- net DDS3_out: track 24.1 -> 23.6 mm
- net DDS4_out: track 31.7 -> 31.2 mm
- net CH4_OUT: track 65.3 -> 65.8 mm
- net P,+15: track 139.1 -> 139.4 mm, vias 7 -> 8
- net ZCEN_DAC: vias 0 -> 1
- net GND: vias 6 -> 10
Other:
- board text removed: "DAC channel 1"
- board text removed: "DAC channel 2"
