File: board/boardv3_morning01112024_final.kicad_pcb (KiCad board)
At the start: 2 copper layers, 92 x 75.8 mm, 69 parts, among them J2 Conn_01x01, J3 Conn_01x01, J3 Conn_01x25_Socket, J4 Conn_01x01, J4 Conn_01x25_Socket, J5 Conn_01x01, J5 PJ-320B, J6 Screw_Terminal_01x02, J7 Screw_Terminal_01x02, J8 Screw_Terminal_01x02

Commit message: hopefully final PCB
Parts:
- removed the G*** at (121.3, 99.5)
- added G***: LOGO, project:logo_negative, F.Cu at (119.2, 100.0)
- C23: moved to B.Cu
- moved C23 0.81 mm to (176.3, 74.5)
Routing:
- net P,-15: track 132.4 -> 127.1 mm, vias 7 -> 8
- net P,+15: track 139.1 -> 141.7 mm
- net CS_AD9833_4: track 57.8 -> 55.7 mm
- net CH2_OUT: track 70.0 -> 70.7 mm
Other:
- board text removed: "DAC channel 1"
- board text removed: "DAC channel 2"
