File: board/board.kicad_sch (KiCad schematic)
At the start: 63 parts, among them J3 Conn_01x25_Socket, J4 Conn_01x25_Socket, J5 PJ-320B, J6 Screw_Terminal_01x02, J7 Screw_Terminal_01x02, J8 Screw_Terminal_01x02

Commit message: hopefully final PCB
Parts:
- removed U13: ~, Package_SO:SOIC-8_3.9x4.9mm_P1.27mm, symbol project:LM258
- added C26: 0.22uF_0603_25V, 4ms_Capacitor:C_0603, symbol 4ms_Capacitor:0.22uF_0603_25V
- added U13: ~, Package_SO:SOIC-8_3.9x4.9mm_P1.27mm, symbol project:OPA227
Connections:
- net +5V: no longer C23.1
- net GND: now also C26.2
- net P,+15: now also C23.1, U13.7 (V+)
- net P,-15: now also C26.1, U13.4 (V-)
- net at R11.2, R13.2, R15.1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: now also U13.3 (In+)
- net at J5.1, J5.2, R8.1: now also U13.6 (Output)
- net at R10.1, R8.2: now also U13.2 (In-)

Commit message: last minute addition (PWM DAC lmao), gerber files,
Parts:
- added R16: 3.0k_0603_0.1%, 4ms_Resistor:R_0603, symbol 4ms_Resistor:3.0k_0603_0.1%
Connections:
- net at R11.2, R13.2, R15.1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: now also R16.2
- net PA8(clock) renamed PWM_DAC_out
- net PWM_DAC_out: now also R16.1
Changed lines of the file:
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@@
 	(wire
 		(pts
+			(xy 220.98 261.62) (xy 220.98 270.51)
+		)
+		(stroke
+			(width 0)
+			(type default)
+		)
+	)
+	(wire
+		(pts
 			(xy 132.08 267.97) (xy 132.08 269.24)
 		)
@@
 		)
 	)
+	(global_label "PWM_DAC_out"
+		(shape input)
+		(at 48.26 162.56 180)
+		(fields_autoplaced yes)
+		(effects
+			(font
+				(size 1.27 1.27)
+			)
+			(justify right)
+		)
+		(property "Intersheetrefs" "${INTERSHEET_REFS}"
+			(at 32.5145 162.56 0)
+			(effects
+				(font
+					(size 1.27 1.27)
+				)
+				(justify right)
+				(hide yes)
+			)
+		)
+	)
 	(global_label "NOISE_TOVOL"
 		(shape input)
@@
 		)
 	)
+	(global_label "PWM_DAC_out"
+		(shape input)
+		(at 213.36 270.51 180)
+		(fields_autoplaced yes)
+		(effects
+			(font
+				(size 1.27 1.27)
+			)
+			(justify right)
+		)
+		(property "Intersheetrefs" "${INTERSHEET_REFS}"
+			(at 197.6145 270.51 0)
+			(effects
+				(font
+					(size 1.27 1.27)
+				)
+				(justify right)
+				(hide yes)
+			)
+		)
+	)
 	(global_label "MUX_SEL_1"
 		(shape input)
@@
 					(unit 1)
 				)
+			)
+		)
+	)
+	(symbol
+		(lib_id "4ms_Resistor:3.0k_0603_0.1%")
+		(at 217.17 270.51 90)
+		(unit 1)
+		(exclude_from_sim no)
+		(in_bom yes)
+		(on_board yes)
+		(dnp no)
+		(fields_autoplaced yes)
+		(property "Reference" "R16"
+			(at 217.17 264.16 90)
+			(effects
+				(font
+					(size 1.27 1.27)
+				)
+			)
+		)
+		(property "Value" "3.0k_0603_0.1%"
+			(at 217.17 273.05 90)
+			(effects
+				(font
+					(size 1.27 1.27)
+				)
+				(hide yes)
+			)
+		)
+		(property "Footprint" "4ms_Resistor:R_0603"
+			(at 229.87 273.05 0)
+			(effects
+				(font
+					(size 1.27 1.27)
+				)
+				(justify left)
+				(hide yes)
+			)
+		)
+		(property "Datasheet" ""
+			(at 217.17 270.51 0)
+			(effects
+				(font
+					(size 1.27 1.27)
+				)
+				(hide yes)
+			)
+		)
+		(property "Description" "3.0k, 0.1%, 1/16W, 0603"
+			(at 217.17 270.51 0)
+			(effects
+				(font
+					(size 1.27 1.27)
+				)
+				(hide yes)
+			)
+		)
+		(property "Specifications" "3.0k, 0.1%, 1/16W, 0603"
+			(at 225.044 273.05 0)
+			(effects
+				(font
+					(size 1.27 1.27)
+				)
+				(justify left)
+				(hide yes)
+			)
+		)
+		(property "Manufacturer" "Vishay / Dale"
+			(at 226.568 273.05 0)
+			(effects
+				(font
+					(size 1.27 1.27)
+				)
+				(justify left)
+				(hide yes)
+			)
+		)
+		(property "Part Number" "TNPW06033K00BEEA"
+			(at 228.092 273.05 0)
+			(effects
+				(font
+					(size 1.27 1.27)
+				)
+				(justify left)
+				(hide yes)
+			)
+		)
+		(property "Display" "3.0k 0.1%"
+			(at 217.17 266.7 90)
+			(effects
+				(font
+					(size 1.27 1.27)
+				)
+			)
+		)
+		(property "JLCPCB ID" "C126481"
+			(at 217.17 270.51 0)
+			(effects
+				(font
+					(size 1.27 1.27)
+				)
+				(hide yes)
+			)
+		)
+		(pin "2"
+		)
+		(pin "1"
+		)
+		(instances
+			(project "board"
+				(path "/e8cec806-e837-4d6f-b166-2de75a563bd6"
+					(reference "R16")
+					(unit 1)
+				)
